File: kad/6502.toy.glue1.kicad_sch (KiCad schematic)
At the start: 9 parts, among them U10 74LS10, U11 74LS30, U12 74LS393, U13 74LS74, U17 74HC00, U19 74HC00, U20 74HC74, U22 74HC138, U8 74LS10

Commit message: update kicad files
Parts:
- added U21: 74HC00, symbol 74xx:74HC00
- added U27: 74HC74, symbol 74xx:74HC74
Connections:
- net A08: now also U21.1, U21.2; no longer U11.12
- net /RD renamed /MRD
- net /WR renamed /MWR
- new net: U11.12, U21.3
Other:
- moved on the sheet: U10B, U10C, U17C
