File: kad/6502.toy.glue2.kicad_sch (KiCad schematic)
At the start: 8 parts, among them U17 74HC00, U19 74HC00, U20 74HC74, U23 74LS00, U24 74LS10, U25 74HC138, U26 74LS00, U9 74LS10

Commit message: update kicad files
Other:
- moved on the sheet: U25
Changed lines of the file:
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@@
 	(symbol
 		(lib_id "74xx:74HC138")
-		(at 213.36 38.1 0)
+		(at 111.76 88.9 0)
 		(unit 1)
 		(exclude_from_sim no)
@@
 		(fields_autoplaced yes)
 		(property "Reference" "U25"
-			(at 215.5033 20.32 0)
+			(at 113.9033 71.12 0)
 			(effects
 				(font
@@
 		)
 		(property "Value" "74HC138"
-			(at 215.5033 22.86 0)
+			(at 113.9033 73.66 0)
 			(effects
 				(font
@@
 		)
 		(property "Footprint" ""
-			(at 213.36 38.1 0)
+			(at 111.76 88.9 0)
 			(effects
 				(font
@@
 		)
 		(property "Datasheet" "http://www.ti.com/lit/ds/symlink/cd74hc238.pdf"
-			(at 213.36 38.1 0)
+			(at 111.76 88.9 0)
 			(effects
 				(font
@@
 		)
 		(property "Description" "3-to-8 line decoder/multiplexer inverting, DIP-16/SOIC-16/SSOP-16"
-			(at 213.36 38.1 0)
+			(at 111.76 88.9 0)
 			(effects
 				(font
